File: hw/frontpanel_dev_adapter/power.sch (KiCad schematic (older format))
At the start: 44 parts, among them J201 KLD-0202-A, J202 Conn_WR-FAST_01x04, J203 Molex_MicroFit_30-43045-0421, Q201 AO4407A, U201 TPS54332DDA, U202 TLV1117LV30DCY, U203 TLV1117LV30DCY

Commit message: FP adapter board: Added LCSC partnumbers to all components to be PnP:ed; Finalized some silk additions; Generated Gerbers, BoM & pnp-files for JCL assembly
Parts:
- C201, C214: LCSC (none) -> C14663
- C202, C203: LCSC (none) -> C15850
- C205, C206, C207, C212, C213, C218, C219: LCSC (none) -> C19702
- C208: LCSC (none) -> C1596
- C209: LCSC (none) -> C32949
- C210: LCSC (none) -> C26404
- C215, C217: footprint Capacitor_SMD:C_0603_1608Metric -> Capacitor_SMD:C_0805_2012Metric; LCSC (none) -> C15850
- D201: LCSC (none) -> C40326
- D202, D203: LCSC (none) -> C72038
- D204, D205, D206: LCSC (none) -> C72043
- Q201: LCSC (none) -> C16072
- R201: LCSC (none) -> C23150
- R202, R204, R206, R207: LCSC (none) -> C25744
- R203: LCSC (none) -> C36871
- R205: LCSC (none) -> C4177
- R208: LCSC (none) -> C25879
- R209, R210: LCSC (none) -> C11702
- U201: LCSC (none) -> C41312
- U202, U203: LCSC (none) -> C15578
Changed lines of the file:
@@
 F 2 "Capacitor_SMD:CP_Elec_6.3x5.8" H 3250 4650 50  0001 C CNN
 F 3 "https://www.mouser.se/datasheet/2/293/e-ucl-1513103.pdf" H 3250 4650 50  0001 C CNN
+F 4 "" H 3250 4650 50  0001 C CNN "LCSCa"
 	1    3250 4650
 	1    0    0    -1
@@
 F 2 "Capacitor_SMD:C_0603_1608Metric" H 2400 4650 50  0001 C CNN
 F 3 "~" H 2400 4650 50  0001 C CNN
+F 4 "C14663" H 2400 4650 50  0001 C CNN "LCSC"
 	1    2400 4650
 	1    0    0    -1
@@
 F 2 "Capacitor_SMD:C_0805_2012Metric" H 3650 1950 50  0001 C CNN
 F 3 "~" H 3650 1950 50  0001 C CNN
+F 4 "C15850" H 3650 1950 50  0001 C CNN "LCSC"
 	1    3650 1950
 	1    0    0    -1
@@
 F 2 "Capacitor_SMD:C_0805_2012Metric" H 4150 1950 50  0001 C CNN
 F 3 "~" H 4150 1950 50  0001 C CNN
+F 4 "C15850" H 4150 1950 50  0001 C CNN "LCSC"
 	1    4150 1950
 	1    0    0    -1
@@
 F 2 "Resistor_SMD:R_0603_1608Metric" H 4650 1650 50  0001 C CNN
 F 3 "~" H 4650 1650 50  0001 C CNN
+F 4 "C23150" H 4650 1650 50  0001 C CNN "LCSC"
 	1    4650 1650
 	1    0    0    -1
@@
 F 2 "Resistor_SMD:R_0402_1005Metric" H 4650 2050 50  0001 C CNN
 F 3 "~" H 4650 2050 50  0001 C CNN
+F 4 "C36871" H 4650 2050 50  0001 C CNN "LCSC"
 	1    4650 2050
 	1    0    0    -1
@@
 F 2 "Capacitor_SMD:C_0603_1608Metric" H 5250 2050 50  0001 C CNN
 F 3 "~" H 5250 2050 50  0001 C CNN
+F 4 "C1596" H 5250 2050 50  0001 C CNN "LCSC"
 	1    5250 2050
 	1    0    0    -1
@@
 F 2 "Capacitor_SMD:C_0402_1005Metric" H 5650 2050 50  0001 C CNN
 F 3 "~" H 5650 2050 50  0001 C CNN
+F 4 "C32949" H 5650 2050 50  0001 C CNN "LCSC"
 	1    5650 2050
 	1    0    0    -1
@@
 F 2 "Resistor_SMD:R_0402_1005Metric" H 6050 2050 50  0001 C CNN
 F 3 "~" H 6050 2050 50  0001 C CNN
+F 4 "C25744" H 6050 2050 50  0001 C CNN "LCSC"
 	1    6050 2050
 	1    0    0    -1
@@
 F 2 "Package_SO:TI_SO-PowerPAD-8_ThermalVias" H 8050 1300 50  0001 C CNN
 F 3 "https://www.ti.com/lit/gpn/tps54332" H 8150 1200 50  0001 C CNN
+F 4 "C41312" H 7150 1650 50  0001 C CNN "LCSC"
 	1    7150 1650
 	1    0    0    -1
@@
 F 2 "Capacitor_SMD:C_0603_1608Metric" H 7850 1450 50  0001 C CNN
 F 3 "~" H 7850 1450 50  0001 C CNN
+F 4 "C14663" V 7850 1450 50  0001 C CNN "LCSC"
 	1    7850 1450
 	0    1    1    0
@@
 F 2 "Resistor_SMD:R_0603_1608Metric" H 8850 2350 50  0001 C CNN
 F 3 "~" H 8850 2350 50  0001 C CNN
+F 4 "C4177" H 8850 2350 50  0001 C CNN "LCSC"
 	1    8850 2350
 	1    0    0    -1
@@
 F 2 "Resistor_SMD:R_0402_1005Metric" H 8850 1950 50  0001 C CNN
 F 3 "~" H 8850 1950 50  0001 C CNN
+F 4 "C25744" H 8850 1950 50  0001 C CNN "LCSC"
 	1    8850 1950
 	1    0    0    -1
@@
 F 2 "customlib_mj_fp:MBRS3xx_SMC_CASE_403AC" H 8150 1675 50  0001 C CNN
 F 3 "https://www.onsemi.com/pub/Collateral/MBRS340T3-D.PDF" H 8150 1850 50  0001 C CNN
+F 4 "C40326" V 8150 1850 50  0001 C CNN "LCSC"
 	1    8150 1850
 	0    1    1    0
@@
 F 2 "customlib_mj_fp:ASPI-0603LR" V 8550 1650 50  0001 C CNN
 F 3 "https://www.mouser.se/datasheet/2/3/ASPI-0630LR-1774844.pdf" V 8550 1650 50  0001 C CNN
+F 4 "" H 8550 1650 50  0001 C CNN "LCSC"
 	1    8550 1650
 	1    0    0    -1
@@
 F 2 "Capacitor_SMD:C_0603_1608Metric" H 9800 1950 50  0001 C CNN
 F 3 "~" H 9800 1950 50  0001 C CNN
+F 4 "C19702" H 9800 1950 50  0001 C CNN "LCSC"
 	1    9800 1950
 	1    0    0    -1
@@
 F 2 "Package_TO_SOT_SMD:SOT-223-3_TabPin2" H 5500 4950 50  0001 C CNN
 F 3 "https://www.ti.com/lit/gpn/tlv1117lv" H 5500 5150 50  0001 C CNN
+F 4 "C15578" H 5500 5150 50  0001 C CNN "LCSC"
 	1    5500 5150
 	1    0    0    -1
@@
 F 2 "Capacitor_SMD:C_0603_1608Metric" H 5000 5350 50  0001 C CNN
 F 3 "~" H 5000 5350 50  0001 C CNN
+F 4 "C19702" H 5000 5350 50  0001 C CNN "LCSC"
 	1    5000 5350
 	1    0    0    -1
@@
 F 2 "Capacitor_SMD:C_0603_1608Metric" H 5900 5350 50  0001 C CNN
 F 3 "~" H 5900 5350 50  0001 C CNN
+F 4 "C19702" H 5900 5350 50  0001 C CNN "LCSC"
 	1    5900 5350
 	1    0    0    -1
@@
 F 2 "LED_SMD:LED_0603_1608Metric" V 1000 6700 50  0001 C CNN
 F 3 "~" V 1000 6700 50  0001 C CNN
+F 4 "C72038" V 1000 6700 50  0001 C CNN "LCSC"
 	1    1000 6700
 	0    -1   -1   0
@@
 F 2 "Resistor_SMD:R_0402_1005Metric" H 1000 6300 50  0001 C CNN
 F 3 "~" H 1000 6300 50  0001 C CNN
+F 4 "C25744" H 1000 6300 50  0001 C CNN "LCSC"
 	1    1000 6300
 	1    0    0    -1
@@
 F 2 "Resistor_SMD:R_0402_1005Metric" H 2000 6300 50  0001 C CNN
 F 3 "~" H 2000 6300 50  0001 C CNN
+F 4 "C25879" H 2000 6300 50  0001 C CNN "LCSC"
 	1    2000 6300
 	1    0    0    -1
@@
 F 2 "Resistor_SMD:R_0402_1005Metric" H 3500 6300 50  0001 C CNN
 F 3 "~" H 3500 6300 50  0001 C CNN
+F 4 "C11702" H 3500 6300 50  0001 C CNN "LCSC"
 	1    3500 6300
 	1    0    0    -1
@@
 F 2 "LED_SMD:LED_0603_1608Metric" V 2000 6700 50  0001 C CNN
 F 3 "~" V 2000 6700 50  0001 C CNN
+F 4 "C72043" V 2000 6700 50  0001 C CNN "LCSC"
 	1    2000 6700
 	0    -1   -1   0
@@
 F 2 "LED_SMD:LED_0603_1608Metric" V 3500 6700 50  0001 C CNN
 F 3 "~" V 3500 6700 50  0001 C CNN
+F 4 "C72043" V 3500 6700 50  0001 C CNN "LCSC"
 	1    3500 6700
 	0    -1   -1   0
@@
 F 2 "Package_TO_SOT_SMD:SOT-223-3_TabPin2" H 5450 3600 50  0001 C CNN
 F 3 "https://www.ti.com/lit/gpn/tlv1117lv" H 5450 3800 50  0001 C CNN
+F 4 "C15578" H 5450 3800 50  0001 C CNN "LCSC"
 	1    5450 3800
 	1    0    0    -1
@@
 F 2 "Capacitor_SMD:C_0603_1608Metric" H 4950 4000 50  0001 C CNN
 F 3 "~" H 4950 4000 50  0001 C CNN
+F 4 "C19702" H 4950 4000 50  0001 C CNN "LCSC"
 	1    4950 4000
 	1    0    0    -1
@@
 F 2 "Capacitor_SMD:C_0603_1608Metric" H 5850 4000 50  0001 C CNN
 F 3 "~" H 5850 4000 50  0001 C CNN
+F 4 "C19702" H 5850 4000 50  0001 C CNN "LCSC"
 	1    5850 4000
 	1    0    0    -1
@@
 F 2 "Resistor_SMD:R_0402_1005Metric" H 3950 6300 50  0001 C CNN
 F 3 "~" H 3950 6300 50  0001 C CNN
+F 4 "C11702" H 3950 6300 50  0001 C CNN "LCSC"
 	1    3950 6300
 	1    0    0    -1
@@
 F 2 "LED_SMD:LED_0603_1608Metric" V 3950 6700 50  0001 C CNN
 F 3 "~" V 3950 6700 50  0001 C CNN
+F 4 "C72043" V 3950 6700 50  0001 C CNN "LCSC"
 	1    3950 6700
 	0    -1   -1   0
@@
 F 0 "C215" H 2850 4750 50  0000 L CNN
 F 1 "10u/16V" H 2800 4550 50  0000 L CNN
-F 2 "Capacitor_SMD:C_0603_1608Metric" H 2800 4650 50  0001 C CNN
+F 2 "Capacitor_SMD:C_0805_2012Metric" H 2800 4650 50  0001 C CNN
 F 3 "~" H 2800 4650 50  0001 C CNN
+F 4 "C15850" H 2800 4650 50  0001 C CNN "LCSC"
 	1    2800 4650
 	1    0    0    -1
@@
 F 2 "Capacitor_SMD:C_0402_1005Metric" H 6050 2350 50  0001 C CNN
 F 3 "~" H 6050 2350 50  0001 C CNN
+F 4 "C26404" H 6050 2350 50  0001 C CNN "LCSC"
 	1    6050 2350
 	1    0    0    -1
@@
 F 2 "Capacitor_SMD:C_0603_1608Metric" H 10250 1950 50  0001 C CNN
 F 3 "~" H 10250 1950 50  0001 C CNN
+F 4 "C19702" H 10250 1950 50  0001 C CNN "LCSC"
 	1    10250 1950
 	1    0    0    -1
@@
 F 2 "Capacitor_SMD:C_0603_1608Metric" H 10650 1950 50  0001 C CNN
 F 3 "~" H 10650 1950 50  0001 C CNN
+F 4 "C19702" H 10650 1950 50  0001 C CNN "LCSC"
 	1    10650 1950
 	1    0    0    -1
@@
 F 2 "LED_SMD:LED_0603_1608Metric" V 600 6700 50  0001 C CNN
 F 3 "~" V 600 6700 50  0001 C CNN
+F 4 "C72038" V 600 6700 50  0001 C CNN "LCSC"
 	1    600  6700
 	0    -1   -1   0
@@
 F 2 "Resistor_SMD:R_0402_1005Metric" H 600 6300 50  0001 C CNN
 F 3 "~" H 600 6300 50  0001 C CNN
+F 4 "C25744" H 600 6300 50  0001 C CNN "LCSC"
 	1    600  6300
 	1    0    0    -1
@@
 F 0 "C217" H 1150 4950 50  0000 L CNN
 F 1 "10u/16V" H 1100 4750 50  0000 L CNN
-F 2 "Capacitor_SMD:C_0603_1608Metric" H 1100 4850 50  0001 C CNN
+F 2 "Capacitor_SMD:C_0805_2012Metric" H 1100 4850 50  0001 C CNN
 F 3 "~" H 1100 4850 50  0001 C CNN
+F 4 "C15850" H 1100 4850 50  0001 C CNN "LCSC"
 	1    1100 4850
 	1    0    0    -1
@@
 F 2 "customlib_mj_fp:SOIC-8_3.9x4.9mm_P1.27mm" H 2250 4425 50  0001 L CIN
 F 3 "https://datasheet.lcsc.com/szlcsc/Alpha-Omega-Semicon-AOS-AO4407A_C16072.pdf" H 2050 4500 50  0001 L CNN
+F 4 "C16072" V 2050 4500 50  0001 C CNN "LCSC"
 	1    2050 4500
 	0    -1   -1   0
