File: hw/ss_debug_adapter/ss_debug_adapter.kicad_pcb (KiCad board)
At the start: 2 copper layers, 50 x 100 mm, 67 parts, among them J101 IDC_2x5, J102 STX-3501-3N_(TTL-232R-xV-AJ), J103 JLink 20-pin IDC, J104 microUSB_5p, J105 Conn_01x04, J106 Conn_01x02, Q101 S9013, Q102 AO3400A, SW101 Pushbutton_SMD_TS-1102W-4316, SW102 Pushbutton_SMD_TS-1102W-4316, U101 STM32F103CBTx, U102 SRV05-4, U103 AMS1117-3.3, U104 TXB0108PWR

Commit message: Kicad 6.0 : Most of SS2k & subprojects updated to kicad6 The projects should from now on be opened through the .kicad_pro files instead of .pro, etc. NOTE: Kicad 6 is now used. Kicad5 is NOT able to open v6+ files.
Connections:
- net /~USB_RENUMn~ renamed /~{USB_RENUMn}
- net ~DBGLEDn~ renamed ~{DBGLEDn}
- net ~RESETn~ renamed ~{RESETn}
Other:
- net class Default removed
