File: hw/ss_backpanel-mirrored_Al/ss_backpanel-mirrored_Al.kicad_pcb (KiCad board)
At the start: 2 copper layers, 165 x 51.1 mm, 26 parts, among them J101 4mm_banana_socket-LB_I4R_A-pa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, M101 Amphenol_T3437000-DIN7_panel_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, M102 Amphenol_T3437000-DIN7_panel_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, M103 Mech_cutout_IDC_2x5, M104 FN283-1-06_Schaffner_AC-panel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, M105 74980104400-Wurth_RJ45-Panel_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, M106 TE-1734346-Panel_cutout, M107 CUI-UJ2_AH_1_SMT-Panel_cutout, M109 SJ-3571N_CUI_audio_jacket_pan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, M110 SMA_bulkhead_jack_Panel_cutout, M111 Molex_NanoFit-1x02-Panel_cuto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

Commit message: Placeholder 3d-models for rear-panel (w. conns), PSU, Bottom-plate, front-panel (w. conns), outer fp
With these placeholder mech. objects, the build-in 3d view of MB pcb features most of the mechanical
objects that constrain components placements. So 3d-view can be used to quickly check and iterate
placements to avoid 3d collisions, without having to first export MB STEP into FreeCAD and muck around
only to have to repeat again for each iteration
Parts:
- turned M104 to 0 degrees
Changed lines of the file:
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@@
     )
     (pad_to_mask_clearance 0)
+    (aux_axis_origin 150 100)
     (grid_origin 150 100)
     (pcbplotparams
@@
   )
   (footprint "customlib_mj_fp:FN283_panel_cutout-outside_mnt" locked (layer "F.Cu")
-    (at 194 74.5 180)
+    (at 194 74.5)
     (descr "Panel cut-outs for Schaffner FN283 AC-inlet")
     (property "Sheetfile" "ss_backpanel-mirrored_Al.kicad_sch")
@@
     (fp_line (start -30 13) (end -30 -13) (layer "Dwgs.User") (width 0.12))
     (fp_line (start 28.5 14.5) (end -28.5 14.5) (layer "Dwgs.User") (width 0.12))
+    (fp_line (start 30 -13) (end 30 13) (layer "Dwgs.User") (width 0.12))
     (fp_line (start -28.5 -14.5) (end 28.5 -14.5) (layer "Dwgs.User") (width 0.12))
-    (fp_line (start 30 -13) (end 30 13) (layer "Dwgs.User") (width 0.12))
-    (fp_arc (start 30 13) (mid 29.56066 14.06066) (end 28.5 14.5) (layer "Dwgs.User") (width 0.12))
     (fp_arc (start -30 -13) (mid -29.56066 -14.06066) (end -28.5 -14.5) (layer "Dwgs.User") (width 0.12))
     (fp_arc (start 28.5 -14.5) (mid 29.56066 -14.06066) (end 30 -13) (layer "Dwgs.User") (width 0.12))
+    (fp_arc (start 30 13) (mid 29.56066 14.06066) (end 28.5 14.5) (layer "Dwgs.User") (width 0.12))
     (fp_arc (start -28.5 14.5) (mid -29.56066 14.06066) (end -30 13) (layer "Dwgs.User") (width 0.12))
+    (fp_line (start -28.5 -14.5) (end 28.5 -14.5) (layer "Edge.Cuts") (width 0.12))
     (fp_line (start -30 13) (end -30 -13) (layer "Edge.Cuts") (width 0.12))
     (fp_line (start 28.5 14.5) (end -28.5 14.5) (layer "Edge.Cuts") (width 0.12))
     (fp_line (start 30 -13) (end 30 13) (layer "Edge.Cuts") (width 0.12))
-    (fp_line (start -28.5 -14.5) (end 28.5 -14.5) (layer "Edge.Cuts") (width 0.12))
     (fp_arc (start -30 -13) (mid -29.56066 -14.06066) (end -28.5 -14.5) (layer "Edge.Cuts") (width 0.12))
+    (fp_arc (start 30 13) (mid 29.56066 14.06066) (end 28.5 14.5) (layer "Edge.Cuts") (width 0.12))
     (fp_arc (start -28.5 14.5) (mid -29.56066 14.06066) (end -30 13) (layer "Edge.Cuts") (width 0.12))
     (fp_arc (start 28.5 -14.5) (mid 29.56066 -14.06066) (end 30 -13) (layer "Edge.Cuts") (width 0.12))
-    (fp_arc (start 30 13) (mid 29.56066 14.06066) (end 28.5 14.5) (layer "Edge.Cuts") (width 0.12))
-    (pad "" np_thru_hole circle locked (at 0 -20 180) (size 3 3) (drill 3) (layers *.Cu *.Mask))
-    (pad "" np_thru_hole circle locked (at 0 20 180) (size 3 3) (drill 3) (layers *.Cu *.Mask))
-    (model "/home/mjoh/projects/stm32/projects/customlib_mj/3d_models/Schaffner-FN283-1-06.stp"
-      (offset (xyz -18 0 19.7))
-      (scale (xyz 1 1 1))
-      (rotate (xyz 0 180 90))
+    (pad "" np_thru_hole circle locked (at 0 -20) (size 3 3) (drill 3) (layers *.Cu *.Mask))
+    (pad "" np_thru_hole circle locked (at 0 20) (size 3 3) (drill 3) (layers *.Cu *.Mask))
+    (model "${KICUSTOMLIB_DIR}/3d_models/AC_Schaffner_inlet_with_QC_sockets.step"
+      (offset (xyz 18 0 19.5))
+      (scale (xyz 1 1 1))
+      (rotate (xyz 0 180 0))
     )
   )
@@
     )
     (pad "" np_thru_hole circle locked (at 0 0) (size 8.3 8.3) (drill 8.3) (layers *.Cu *.Mask))
-    (model "/home/mjoh/projects/stm32/projects/customlib_mj/3d_models/LB_I4R_A-black.stp"
+    (model "${KICUSTOMLIB_DIR}/3d_models/4mmBanana_panel_with_QC.step"
       (offset (xyz 0 0 -20.5))
       (scale (xyz 1 1 1))
-      (rotate (xyz -90 0 90))
-    )
-  )
+      (rotate (xyz 180 0 0))
+    )
+  )
